Commit message: add ROS2 branch of CHAMP with ament_cmake, teleop, and robot configs

File: ros2/champ_description/urdf/accessories.urdf.xacro (robot description, xacro)
@@ -2,6 +2,6 @@
 <robot xmlns:xacro="http://ros.org/wiki/xacro">
     <xacro:macro name="accessories" params="base_name base_length base_height  " >
-        <xacro:include filename="$(find hector_sensors_description)/urdf/hokuyo_utm30lx.urdf.xacro" />
-        <xacro:include filename="$(find hector_sensors_description)/urdf/asus_camera.urdf.xacro" />
+        <xacro:include filename="$(find champ_description)/urdf/hokuyo_utm30lx.urdf.xacro" />
+        <xacro:include filename="$(find champ_description)/urdf/asus_camera.urdf.xacro" />
         <xacro:hokuyo_utm30lx
             name="hokuyo"
@@ -19,17 +19,4 @@
             <origin xyz="${base_length / 2} 0.0 -${base_height / 2 + 0.01}" rpy="0 0 0"/>
         </xacro:asus_camera>
-        <gazebo>
-            <plugin name="imu_controller" filename="libhector_gazebo_ros_imu.so">
-                <updateRate>50.0</updateRate>
-                <bodyName>imu_link</bodyName>
-                <topicName>imu/data</topicName>
-                <accelDrift>0.005 0.005 0.005</accelDrift>
-                <accelGaussianNoise>0.005 0.005 0.005</accelGaussianNoise>
-                <rateDrift>0.005 0.005 0.005 </rateDrift>
-                <rateGaussianNoise>0.005 0.005 0.005 </rateGaussianNoise>
-                <headingDrift>0.005</headingDrift>
-                <headingGaussianNoise>0.005</headingGaussianNoise>
-            </plugin>
-        </gazebo>
         <link name="imu_link">
             <inertial>
@@ -43,4 +30,25 @@
             <child link="imu_link" />
         </joint>
+        <gazebo reference="imu_link">
+                <sensor name="imu_controller" type="imu">
+                    <always_on>true</always_on>
+                    <update_rate>50</update_rate>
+                    <plugin name="gazebo_ros_imu_sensor" filename="libgazebo_ros_imu_sensor.so">
+                        <ros>
+                            <namespace>/imu</namespace>
+                            <argument>~/out:=data</argument>
+                        </ros>
+                        <!-- <updateRate>50.0</updateRate>
+                        <bodyName>imu_link</bodyName>
+                        <topicName>imu/data</topicName>
+                        <accelDrift>0.005 0.005 0.005</accelDrift>
+                        <accelGaussianNoise>0.005 0.005 0.005</accelGaussianNoise>
+                        <rateDrift>0.005 0.005 0.005 </rateDrift>
+                        <rateGaussianNoise>0.005 0.005 0.005 </rateGaussianNoise>
+                        <headingDrift>0.005</headingDrift>
+                        <headingGaussianNoise>0.005</headingGaussianNoise> -->
+                    </plugin>
+                </sensor>
+            </gazebo>
         <!-- <xacro:include filename="$(find velodyne_description)/urdf/VLP-16.urdf.xacro"/>
         <xacro:VLP-16 parent="${base_name}" name="velodyne" topic="velodyne_points" hz="10" samples="1024" gpu="false" lasers="16" max_range="100">

File: ros2/champ_description/urdf/champ.urdf (robot description, URDF)
Before this commit: robot champ, 29 links, 28 joints
Links:
- link base_link: geometry collision mesh filename=file:///home/Alexander.Karavaev/champ_ws/install/champ_desc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 scale=0.001 0.001 0.001; visual mesh filename=file:///home/Alexander.Karavaev/champ_ws/install/champ_desc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 scale=0.001 0.001 0.001
- link camera_link: geometry collision mesh filename=file:///home/Alexander.Karavaev/champ_ws/install/champ_desc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; visual mesh filename=file:///home/Alexander.Karavaev/champ_ws/install/champ_desc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
- link hokuyo_frame: geometry collision box size=0.058 0.058 0.087; visual mesh filename=file:///home/Alexander.Karavaev/champ_ws/install/champ_desc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
- link lf_hip_link: geometry collision mesh filename=file:///home/Alexander.Karavaev/champ_ws/install/champ_desc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 scale=0.001 0.001 0.001; visual mesh filename=file:///home/Alexander.Karavaev/champ_ws/install/champ_desc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 scale=0.001 0.001 0.001
- link lf_lower_leg_link: geometry collision mesh filename=file:///home/Alexander.Karavaev/champ_ws/install/champ_desc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 scale=0.001 0.001 0.001; visual mesh filename=file:///home/Alexander.Karavaev/champ_ws/install/champ_desc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 scale=0.001 0.001 0.001
- link lf_upper_leg_link: geometry collision mesh filename=file:///home/Alexander.Karavaev/champ_ws/install/champ_desc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 scale=0.001 0.001 0.001; visual mesh filename=file:///home/Alexander.Karavaev/champ_ws/install/champ_desc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 scale=0.001 0.001 0.001
- link lh_hip_link: geometry collision mesh filename=file:///home/Alexander.Karavaev/champ_ws/install/champ_desc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 scale=0.001 0.001 0.001; visual mesh filename=file:///home/Alexander.Karavaev/champ_ws/install/champ_desc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 scale=0.001 0.001 0.001
- link lh_lower_leg_link: geometry collision mesh filename=file:///home/Alexander.Karavaev/champ_ws/install/champ_desc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 scale=0.001 0.001 0.001; visual mesh filename=file:///home/Alexander.Karavaev/champ_ws/install/champ_desc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 scale=0.001 0.001 0.001
- link lh_upper_leg_link: geometry collision mesh filename=file:///home/Alexander.Karavaev/champ_ws/install/champ_desc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 scale=0.001 0.001 0.001; visual mesh filename=file:///home/Alexander.Karavaev/champ_ws/install/champ_desc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 scale=0.001 0.001 0.001
- link rf_hip_link: geometry collision mesh filename=file:///home/Alexander.Karavaev/champ_ws/install/champ_desc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 scale=0.001 0.001 0.001; visual mesh filename=file:///home/Alexander.Karavaev/champ_ws/install/champ_desc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 scale=0.001 0.001 0.001
- link rf_lower_leg_link: geometry collision mesh filename=file:///home/Alexander.Karavaev/champ_ws/install/champ_desc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 scale=0.001 0.001 0.001; visual mesh filename=file:///home/Alexander.Karavaev/champ_ws/install/champ_desc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 scale=0.001 0.001 0.001
- link rf_upper_leg_link: geometry collision mesh filename=file:///home/Alexander.Karavaev/champ_ws/install/champ_desc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 scale=0.001 0.001 0.001; visual mesh filename=file:///home/Alexander.Karavaev/champ_ws/install/champ_desc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 scale=0.001 0.001 0.001
- link rh_hip_link: geometry collision mesh filename=file:///home/Alexander.Karavaev/champ_ws/install/champ_desc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 scale=0.001 0.001 0.001; visual mesh filename=file:///home/Alexander.Karavaev/champ_ws/install/champ_desc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 scale=0.001 0.001 0.001
- link rh_lower_leg_link: geometry collision mesh filename=file:///home/Alexander.Karavaev/champ_ws/install/champ_desc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 scale=0.001 0.001 0.001; visual mesh filename=file:///home/Alexander.Karavaev/champ_ws/install/champ_desc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 scale=0.001 0.001 0.001
- link rh_upper_leg_link: geometry collision mesh filename=file:///home/Alexander.Karavaev/champ_ws/install/champ_desc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 scale=0.001 0.001 0.001; visual mesh filename=file:///home/Alexander.Karavaev/champ_ws/install/champ_desc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 scale=0.001 0.001 0.001
Joints:
- joint camera_depth_optical_joint: origin xyz=0 0 0 rpy=-1.57079632679 0.0 -1.57079632679 -> xyz=0 0 0 rpy=-1.5707963267948966 0.0 -1.5707963267948966
- joint camera_rgb_optical_joint: origin xyz=0 0 0 rpy=-1.57079632679 0.0 -1.57079632679 -> xyz=0 0 0 rpy=-1.5707963267948966 0.0 -1.5707963267948966
- joint hokuyo_joint: origin xyz=0.0 0.0 0.105 rpy=0 0 0 -> xyz=0.0 0.0 0.10500000000000001 rpy=0 0 0
- joint lf_foot_joint: origin xyz=0 0 -0.141 rpy=0 0 0 -> xyz=0.00325 0 -0.141 rpy=0 0 0
- joint lf_hip_joint: limit lower=-3.14159265359 upper=3.14159265359 effort=25 velocity=1.5 -> lower=-3.141592653589793 upper=3.141592653589793 effort=25 velocity=1.5
- joint lf_lower_leg_joint: limit lower=-3.14159265359 upper=3.14159265359 effort=25 velocity=1.5 -> lower=-3.141592653589793 upper=3.141592653589793 effort=25 velocity=1.5
- joint lf_upper_leg_joint: limit lower=-3.14159265359 upper=3.14159265359 effort=25 velocity=1.5 -> lower=-3.141592653589793 upper=3.141592653589793 effort=25 velocity=1.5
- joint lh_foot_joint: origin xyz=0 0 -0.141 rpy=0 0 0 -> xyz=0.00325 0 -0.141 rpy=0 0 0
- joint lh_hip_joint: limit lower=-3.14159265359 upper=3.14159265359 effort=25 velocity=1.5 -> lower=-3.141592653589793 upper=3.141592653589793 effort=25 velocity=1.5
- joint lh_lower_leg_joint: limit lower=-3.14159265359 upper=3.14159265359 effort=25 velocity=1.5 -> lower=-3.141592653589793 upper=3.141592653589793 effort=25 velocity=1.5
- joint lh_upper_leg_joint: limit lower=-3.14159265359 upper=3.14159265359 effort=25 velocity=1.5 -> lower=-3.141592653589793 upper=3.141592653589793 effort=25 velocity=1.5
- joint rf_foot_joint: origin xyz=0 0 -0.141 rpy=0 0 0 -> xyz=0.00325 0 -0.141 rpy=0 0 0
- joint rf_hip_joint: limit lower=-3.14159265359 upper=3.14159265359 effort=25 velocity=1.5 -> lower=-3.141592653589793 upper=3.141592653589793 effort=25 velocity=1.5
- joint rf_lower_leg_joint: limit lower=-3.14159265359 upper=3.14159265359 effort=25 velocity=1.5 -> lower=-3.141592653589793 upper=3.141592653589793 effort=25 velocity=1.5
- joint rf_upper_leg_joint: limit lower=-3.14159265359 upper=3.14159265359 effort=25 velocity=1.5 -> lower=-3.141592653589793 upper=3.141592653589793 effort=25 velocity=1.5
- joint rh_foot_joint: origin xyz=0 0 -0.141 rpy=0 0 0 -> xyz=0.00325 0 -0.141 rpy=0 0 0
- joint rh_hip_joint: limit lower=-3.14159265359 upper=3.14159265359 effort=25 velocity=1.5 -> lower=-3.141592653589793 upper=3.141592653589793 effort=25 velocity=1.5
- joint rh_lower_leg_joint: limit lower=-3.14159265359 upper=3.14159265359 effort=25 velocity=1.5 -> lower=-3.141592653589793 upper=3.141592653589793 effort=25 velocity=1.5
- joint rh_upper_leg_joint: limit lower=-3.14159265359 upper=3.14159265359 effort=25 velocity=1.5 -> lower=-3.141592653589793 upper=3.141592653589793 effort=25 velocity=1.5

File: ros2/champ_description/urdf/champ.urdf.xacro (robot description, xacro)
@@ -13,5 +13,5 @@
             <origin xyz="0 0 0" rpy="0 0 0" />
             <geometry>
-                <mesh filename="package://champ_description/meshes/base.stl" scale="0.001 0.001 0.001" />
+                <mesh filename="file://$(find champ_description)/meshes/base_simple.stl" scale="0.001 0.001 0.001" />
             </geometry>
             <material name="black" />
@@ -32,4 +32,9 @@
         <origin rpy="0 0 0" xyz="0 0 0"/>
     </joint>
+    <!-- <link name="world"/>
+    <joint name="fixed" type="fixed">
+        <parent link="world"/>
+        <child link="base_link"/>
+      </joint> -->
     <gazebo reference="base_link">
         <material>Gazebo/FlatBlack</material>
@@ -48,18 +53,19 @@
     <gazebo>
       <plugin name="p3d_base_controller" filename="libgazebo_ros_p3d.so">
-            <alwaysOn>true</alwaysOn>
-            <updateRate>10.0</updateRate>
-            <bodyName>base_link</bodyName>
-            <topicName>odom/ground_truth</topicName>
-            <gaussianNoise>0.01</gaussianNoise>
-            <frameName>world</frameName>
-            <xyzOffsets>0 0 0</xyzOffsets>
-            <rpyOffsets>0 0 0</rpyOffsets>
-        </plugin>
+        <ros>
+            <argument>odom:=odom/ground_truth</argument>
+        </ros>
+        <body_name>base_link</body_name>
+        <frame_name>world</frame_name>
+        <update_rate>10.0</update_rate>
+        <xyz_offset>0 0 0</xyz_offset>
+        <rpy_offset>0 0 0</rpy_offset>
+        <gaussian_noise>0.01</gaussian_noise>
+    </plugin>
     </gazebo>
     <gazebo>
-        <plugin name="gazebo_ros_control" filename="libgazebo_ros_control.so">
-            <legacyModeNS>true</legacyModeNS>
-        </plugin>
+        <plugin filename="libgazebo_ros2_control.so" name="gazebo_ros2_control">
+        <parameters>$(find champ_gazebo)/config/ros_control.yaml</parameters>
+      </plugin>
     </gazebo>
 </robot>

File: ros2/champ_description/urdf/leg.urdf.xacro (robot description, xacro)
@@ -91,13 +91,13 @@
         </link>
         <gazebo reference="${leg}_lower_leg_link">
-            <kp>1000000.0</kp>
-            <kd>1.0</kd>
+            <kp>10000000000.0</kp>
+            <kd>100.0</kd>
             <mu1>0.8</mu1>
             <mu2>0.8</mu2>
-            <maxVel>0.0</maxVel>
-            <minDepth>0.001</minDepth>
+            <minDepth>0.05</minDepth>
             <material>Gazebo/FlatBlack</material>
         </gazebo>
         <link name="${leg}_foot_link" />
+        <!-- <link name="${leg}_foot_link_debug" /> -->
         <joint name="${leg}_debug_joint" type="fixed">
             <parent link="base_link" />
@@ -129,37 +129,32 @@
             <parent link="${leg}_lower_leg_link" />
             <child link="${leg}_foot_link" />
-            <!-- <origin xyz="0.00325 0 -${lower_leg_to_foot_distance}" rpy="0 0 0" /> -->
-            <origin xyz="0 0 -${lower_leg_to_foot_distance}" rpy="0 0 0" />
+            <origin xyz="0.00325 0 -${lower_leg_to_foot_distance}" rpy="0 0 0" />
+            <!-- <origin xyz="0 0 -${lower_leg_to_foot_distance}" rpy="0 0 0" /> -->
         </joint>
-        <transmission name="${leg}_hip_joint_trans">
-            <type>transmission_interface/SimpleTransmission</type>
+        <!-- <joint name="${leg}_debug_joint_foot" type="fixed">
+            <parent link="${leg}_foot_link" />
+            <child link="${leg}_foot_link_debug" />
+            <origin xyz="0 0 0" rpy="0 0 0" />
+        </joint> -->
+        <ros2_control name="${leg}" type="system">
+            <hardware>
+                <plugin>gazebo_ros2_control/GazeboSystem</plugin>
+            </hardware>
             <joint name="${leg}_hip_joint">
-                <hardwareInterface>hardware_interface/EffortJointInterface</hardwareInterface>
+                <command_interface name="effort"/>
+                <state_interface name="position"/>
+                <state_interface name="velocity"/>
             </joint>
-            <actuator name="${leg}_hip_joint_motor">
-                <hardwareInterface>hardware_interface/EffortJointInterface</hardwareInterface>
-                <mechanicalReduction>1</mechanicalReduction>
-            </actuator>
-        </transmission>
-        <transmission name="${leg}_upper_leg_joint_trans">
-            <type>transmission_interface/SimpleTransmission</type>
             <joint name="${leg}_upper_leg_joint">
-                <hardwareInterface>hardware_interface/EffortJointInterface</hardwareInterface>
+                <command_interface name="effort"/>
+                <state_interface name="position"/>
+                <state_interface name="velocity"/>
             </joint>
-            <actuator name="${leg}_upper_leg_joint_motor">
-                <hardwareInterface>hardware_interface/EffortJointInterface</hardwareInterface>
-                <mechanicalReduction>1</mechanicalReduction>
-            </actuator>
-        </transmission>
-        <transmission name="${leg}_lower_leg_joint_trans">
-            <type>transmission_interface/SimpleTransmission</type>
             <joint name="${leg}_lower_leg_joint">
-                <hardwareInterface>hardware_interface/EffortJointInterface</hardwareInterface>
+                <command_interface name="effort"/>
+                <state_interface name="position"/>
+                <state_interface name="velocity"/>
             </joint>
-            <actuator name="${leg}_lower_joint_motor">
-                <hardwareInterface>hardware_interface/EffortJointInterface</hardwareInterface>
-                <mechanicalReduction>1</mechanicalReduction>
-            </actuator>
-        </transmission>
+        </ros2_control>
     </xacro:macro>
 </robot>
