Commit message: Add arm reach/gripper IK control and pick demo

File: ros2/champ_description/urdf/arm.urdf.xacro (robot description, xacro)
@@ -3,7 +3,17 @@
   5-DOF manipulator arm, extracted from the flat champ_arm.urdf dump (CHAMP's
   stock demo arm: base_joint/lower_arm_joint/upper_arm_joint/wrist1_joint/
-  wrist2_joint, no gripper) into a reusable macro so it can be mounted on any
-  robot base link instead of only the generic champ_description/champ.urdf
-  robot it originally shipped hardcoded into.
+  wrist2_joint) into a reusable macro so it can be mounted on any robot base
+  link instead of only the generic champ_description/champ.urdf robot it
+  originally shipped hardcoded into.
+  A simple 2-finger parallel gripper is bolted onto wrist2 below (no STL for
+  it in champ_description/meshes/arm, since CHAMP's stock arm never had one,
+  so it's box primitives instead of a mesh). left_finger_joint is the one
+  driven directly; right_finger_joint carries a <mimic> of it (multiplier
+  -1) for URDF-spec consumers (robot_state_publisher/RViz/MoveIt), but see
+  the caveat on right_finger_joint below: that constraint is NOT enforced in
+  this repo's actual Gazebo control path, so right_finger_joint also gets
+  its own native command topic and must be driven in lockstep with
+  left_finger_joint by whatever commands the gripper (see
+  intelligence/manipulation/arm_reach_node.py).
 -->
 <robot xmlns:xacro="http://ros.org/wiki/xacro">
@@ -156,4 +166,95 @@
       <origin rpy="0 0 0" xyz="0.065 0 0"/>
     </joint>
+    <!-- Parallel gripper. wrist2_to_gripper_joint is fixed, so it just adds
+         a rigid offset to the end effector, kept in sync with
+         intelligence/manipulation/arm_ik.py's GRIPPER_LENGTH constant
+         (wrist2_joint -> fingertip centerline distance = 0.015 + 0.04). -->
+    <link name="gripper_base">
+      <inertial>
+        <origin rpy="0 0 0" xyz="0 0 0"/>
+        <mass value="0.03"/>
+        <inertia ixx="1e-5" ixy="0" ixz="0" iyy="1e-5" iyz="0" izz="1e-5"/>
+      </inertial>
+      <collision>
+        <origin rpy="0 0 0" xyz="0 0 0"/>
+        <geometry>
+          <box size="0.02 0.05 0.02"/>
+        </geometry>
+      </collision>
+      <visual>
+        <origin rpy="0 0 0" xyz="0 0 0"/>
+        <geometry>
+          <box size="0.02 0.05 0.02"/>
+        </geometry>
+        <material name="black"/>
+      </visual>
+    </link>
+    <joint name="wrist2_to_gripper_joint" type="fixed">
+      <parent link="wrist2"/>
+      <child link="gripper_base"/>
+      <origin rpy="0 0 0" xyz="0.015 0 0"/>
+    </joint>
+    <!-- Fingers slide along +/-y from the centerline: joint value 0 = closed,
+         0.025 = fully open (5cm max gap between finger inner faces). -->
+    <link name="left_finger">
+      <inertial>
+        <origin rpy="0 0 0" xyz="0 0 0"/>
+        <mass value="0.01"/>
+        <inertia ixx="1e-6" ixy="0" ixz="0" iyy="1e-6" iyz="0" izz="1e-6"/>
+      </inertial>
+      <collision>
+        <origin rpy="0 0 0" xyz="0 0 0"/>
+        <geometry>
+          <box size="0.03 0.008 0.015"/>
+        </geometry>
+      </collision>
+      <visual>
+        <origin rpy="0 0 0" xyz="0 0 0"/>
+        <geometry>
+          <box size="0.03 0.008 0.015"/>
+        </geometry>
+        <material name="black"/>
+      </visual>
+    </link>
+    <joint name="left_finger_joint" type="prismatic">
+      <axis xyz="0 1 0"/>
+      <limit effort="10" lower="0.0" upper="0.025" velocity="0.5"/>
+      <parent link="gripper_base"/>
+      <child link="left_finger"/>
+      <origin rpy="0 0 0" xyz="0.04 0 0"/>
+    </joint>
+    <link name="right_finger">
+      <inertial>
+        <origin rpy="0 0 0" xyz="0 0 0"/>
+        <mass value="0.01"/>
+        <inertia ixx="1e-6" ixy="0" ixz="0" iyy="1e-6" iyz="0" izz="1e-6"/>
+      </inertial>
+      <collision>
+        <origin rpy="0 0 0" xyz="0 0 0"/>
+        <geometry>
+          <box size="0.03 0.008 0.015"/>
+        </geometry>
+      </collision>
+      <visual>
+        <origin rpy="0 0 0" xyz="0 0 0"/>
+        <geometry>
+          <box size="0.03 0.008 0.015"/>
+        </geometry>
+        <material name="black"/>
+      </visual>
+    </link>
+    <!-- multiplier=-1: right_finger mirrors left_finger's slide so the two
+         close/open symmetrically about the centerline. Not enforced by this
+         repo's Gazebo control path (gz sdf -p's URDF->SDF conversion does
+         not carry <mimic> through), so it's driven directly instead, see
+         the macro-level comment above. -->
+    <joint name="right_finger_joint" type="prismatic">
+      <axis xyz="0 1 0"/>
+      <limit effort="10" lower="-0.025" upper="0.0" velocity="0.5"/>
+      <parent link="gripper_base"/>
+      <child link="right_finger"/>
+      <origin rpy="0 0 0" xyz="0.04 0 0"/>
+      <mimic joint="left_finger_joint" multiplier="-1" offset="0"/>
+    </joint>
   </xacro:macro>
 </robot>

File: urdf/go2_unitree/urdf/go2_gz.urdf (robot description, URDF)
Before this commit: robot go2_description, 35 links, 34 joints
Links:
- added link gripper_base, mass 0.03; collision box size=0.02 0.05 0.02; visual box size=0.02 0.05 0.02
- added link left_finger, mass 0.01; collision box size=0.03 0.008 0.015; visual box size=0.03 0.008 0.015
- added link right_finger, mass 0.01; collision box size=0.03 0.008 0.015; visual box size=0.03 0.008 0.015
Joints:
- added joint left_finger_joint: type prismatic, parent gripper_base, child left_finger, origin xyz=0.04 0 0 rpy=0 0 0, axis 0 1 0, limit lower=0.0 upper=0.025 effort=10 velocity=0.5
- added joint right_finger_joint: type prismatic, parent gripper_base, child right_finger, origin xyz=0.04 0 0 rpy=0 0 0, axis 0 1 0, limit lower=-0.025 upper=0.0 effort=10 velocity=0.5, mimic joint=left_finger_joint multiplier=-1 offset=0
- added joint wrist2_to_gripper_joint: type fixed, parent wrist2, child gripper_base, origin xyz=0.015 0 0 rpy=0 0 0

File: urdf/go2_unitree/urdf/go2_gz.urdf.xacro (robot description, xacro)
@@ -10,9 +10,15 @@
     <origin rpy="0 0 0" xyz="0.08 0 0.057"/>
   </xacro:champ_arm>
-  <!-- Gazebo Harmonic gz_ros2_control plugin -->
+  <!-- Gazebo Harmonic gz_ros2_control plugin. training/ has no package.xml
+       (it's plain Python run via `python3 script.py`, not a ROS2 package),
+       so $(find training) can't resolve it: it previously fell through to
+       whatever other overlaid workspace happened to have a colcon package
+       literally named "training" and baked in that repo's install path.
+       __REPO_ROOT__ is resolved dynamically (to this checkout's actual path)
+       by scripts/make_go2_stand.py when it converts this file to SDF. -->
   <gazebo>
     <plugin filename="libgz_ros2_control-system.so"
             name="gz_ros2_control::GazeboSimROS2ControlPlugin">
-      <parameters>$(find training)/config/go2_ros2_control.yaml</parameters>
+      <parameters>__REPO_ROOT__/training/config/go2_ros2_control.yaml</parameters>
     </plugin>
   </gazebo>
@@ -107,4 +113,17 @@
       <state_interface name="velocity"/>
     </joint>
+    <!-- Both fingers get independent command interfaces, see
+         ros2/champ_description/urdf/arm.urdf.xacro's macro-level comment on
+         why right_finger_joint's <mimic> isn't relied on here. -->
+    <joint name="left_finger_joint">
+      <command_interface name="position"/>
+      <state_interface name="position"><param name="initial_value">0.0</param></state_interface>
+      <state_interface name="velocity"/>
+    </joint>
+    <joint name="right_finger_joint">
+      <command_interface name="position"/>
+      <state_interface name="position"><param name="initial_value">0.0</param></state_interface>
+      <state_interface name="velocity"/>
+    </joint>
   </ros2_control>
   <!-- IMU sensor on base -->
